File: Design/H05R0.brd (EAGLE design)
At the start: 60 x 34.6 mm, 62 parts, among them J1 1984617_MOD, Q1 ECH8693R-TL-W, U1 STM32G0B1CEU6N, U2 MAX17330X22+, U3 TPS631000DRLR, U4 LD39200PU33R, X1 XTALL_CSTCE8M00G52

Commit message: Unreviewed version - update the design by adding additional transistors in parallel.
Parts:
- removed C6: 100nF, HEXABITZ_RCLS:C-0603
- removed C7: 4.7uF, HEXABITZ_RCLS:C-0805-POL
- added Q2: ECH8693R-TL-W, HEXABITZ_RCLS:SOTFL65P280X95-8N
- added U5: NCP45521IMNTWG-LDFN8_2X2_ONS, HEXABITZ_ICs:DFN8_2X2_ONS
- U1: value STM32G0B1CEU6N -> STM32G0B1CEU6QFN_B1CEU6_STM-L; device HEXABITZ_ICs:HEXABITZ_ICS_QFN_B1CEU6_STM-L -> HEXABITZ_ICs:QFN_B1CEU6_STM-L
- moved D4 14.6 mm to (-9.51, 15.0), turned to 180 degrees
- moved R10 3.15 mm to (15.0, 9.02)
- moved R14 1.58 mm to (23.1, 1.88)
- moved FB1 0.79 mm to (-7.45, 14.1), flipped to the bottom
- moved C18 0.57 mm to (15.5, 2.80)
- moved R9 0.39 mm to (14.0, 2.95)
Connections:
- new net N$4: Q2.5, Q2.6, Q2.7, Q2.8
- new net VCC: U5.3
- new net VIN: U5.9
- new net VIN_2: U5.1
- net CSP: now also Q2.1
- net GND: no longer C6.2, C7.2, U1.30
- net N$10: now also Q2.2
- net N$15: now also Q2.4
- net VBUS: now also Q2.3
- net VDD: no longer C6.1, C7.1, U1.31
Routing:
- net GND: track 0.00 -> 92.6 mm
- net VSSA: track 0.00 -> 78.3 mm
- net VDD: track 12.9 -> 85.3 mm, vias 6 -> 5
- net VBUS: track 14.8 -> 32.3 mm, vias 6 -> 9
- net CSP: track 6.98 -> 12.8 mm
- net N$10: track 3.22 -> 7.77 mm, vias 0 -> 2
- net N$15: track 1.74 -> 5.79 mm
- net DIS: track 8.42 -> 11.7 mm
- net USART3_TX: track 11.0 -> 13.1 mm
- net N$17: track 10.6 -> 12.0 mm
- net USART1_TX: track 16.2 -> 15.1 mm
- net VBAT: track 12.1 -> 12.6 mm
- added copper zone on layer 16, net N$4
- removed copper zone on layer 1, net VDDA
Other:
- board text added: "*"
- board text added: "H05R01"
- board text removed: "H05R00"

Commit message: - New version: Schematic finished and reviewed. Other files have not been modified yet for the new design.
Parts:
- removed D2: UCLAMP0501H.TCT, HEXABITZ_RCLS:SODFL1608X70N
- removed J1: 1984617_MOD, HEXABITZ_CONNECTION_PARTS:1984617_MOD
- removed Q2: ECH8693R-TL-W, HEXABITZ_RCLS:SOTFL65P280X95-8N
- removed R1: 0.0R, HEXABITZ_RCLS:R-0603
- added BAT_J2: B2P-VH-FB-B_LF__SN_, HEXABITZ_CONNECTION_PARTS:B2PVHFBBLFSN
- added C19: 10uF, HEXABITZ_RCLS:C-0805
- added C20, C6: 1uF, HEXABITZ_RCLS:C-0805
- added C21, C22, C23: 100nF, HEXABITZ_RCLS:C-0603
- added C24: 22nF, HEXABITZ_RCLS:C-0603
- added C7: 4.7uF, HEXABITZ_RCLS:C-0805
- added PIO_J: 3-644456-2, HEXABITZ_USER_INTERFACE_PARTS:TE_3-644456-2
- added R25, R28: 100K, HEXABITZ_RCLS:R-0603
- added R26, R27: 4.7K, HEXABITZ_RCLS:R-0603
- added R29: 100R, HEXABITZ_RCLS:R-0603
- added R30: 0R, HEXABITZ_RCLS:R-0603
- added SJ1, SJ2: (no value), jumper:SJ
- added U6: LDK130C33R, HEXABITZ_ICs:SOT65P210X110-5N
- added VBUS_OUT_J: 1984617, HEXABITZ_CONNECTION_PARTS:1984617
- Q1: value ECH8693R-TL-W -> SISF06DN-T1-GE3; device HEXABITZ_RCLS:SOTFL65P280X95-8N -> HEXABITZ_ICs:SISF06DNT1GE3
- R4: value 10 mR -> 5 mR
- R5: value 100K -> 33K
- R6: value 665K -> 220K
- U5: value NCP45521IMNTWG-LDFN8_2X2_ONS -> NCP45521IMNTWG-L
- USB_C: value UJC-HP-G-SMT-TR -> 12401610E4#2A; device HEXABITZ_CONNECTION_PARTS:CUI_UJC-HP-G-SMT-TR -> HEXABITZ_CONNECTION_PARTS:12401610E42A
- moved U4 232.8 mm to (-37.6, -218.1)
- moved C16 228.8 mm to (-29.5, -209.4)
- moved C10 227.7 mm to (-43.2, -209.4), turned to 0 degrees
- moved L1 227.2 mm to (-34.4, -214.0), turned to 0 degrees
- moved R5 226.8 mm to (-43.2, -204.9), turned to 0 degrees
- moved C11 226.5 mm to (-38.7, -209.4), turned to 0 degrees
- moved R7 226.1 mm to (-34.0, -204.9), turned to 0 degrees
- moved R6 224.6 mm to (-38.6, -204.9)
- moved C15 223.0 mm to (-34.1, -209.4), turned to 0 degrees
- moved R8 221.5 mm to (-29.4, -204.9), flipped to the top, turned to 0 degrees
- moved R20 219.7 mm to (-24.8, -204.9), flipped to the top, turned to 0 degrees
- moved C9 219.0 mm to (-15.6, -204.9), turned to 0 degrees
- moved U3 202.2 mm to (-29.4, -185.7), turned to 0 degrees
- moved R17 162.9 mm to (-43.2, -148.6)
- moved R15 156.9 mm to (-43.2, -144.0)
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Connections:
- net DIS renamed N$24
- removed net CHG: R9.2, U2.C2
- removed net CSP: C18.1, Q1.1, Q2.1, R4.2, U2.A3
- removed net N$13 (its old number): R20.2, R7.2, U3.6
- removed net N$4: Q2.5, Q2.6, Q2.7, Q2.8
- removed net N$9: Q1.5, Q1.6, Q1.7, Q1.8
- removed net VCC: U5.3
- removed net VIN: U5.9
- removed net VIN_2: U5.1
- removed net VSSA: BAT_J.2, C10.1, C11.1, C13.2, C14.2, C17.1, C2.2, C3.2, C4.2, C5.2, C8.2, C9.1, D2.2, EXT_TH_J.1, J1.2, R1.1, R13.1, R14.1, R19.2, R5.1, R7.1, U1.7, U2.A2, U3.7, U4.7, USB_C.A1, USB_C.A12, USB_C.B1, USB_C.B12, USB_C.S1, USB_C.S2, USB_C.S3, USB_C.S4
- new net 3V3_OUT: C15.2, SJ2.1, U$1.PAD_PU11, U$1.PAD_PU12, U$1.PAD_PU13, U$1.PAD_PU14, U$1.PAD_PU15, U$1.PAD_PU16, U$1.PAD_PU17, U$1.PAD_PU18, U$1.PAD_PU19, U$1.PAD_PU20, U4.1, U4.2
- new net 3V3_OUT_EN: R28.2, U4.5
- new net MCU_3V3: C21.2, C7.1, R11.2, R21.2, R22.2, SJ2.2, U5.3, U6.5
- new net N$16: R8.2, U3.5
- new net N$22: R25.1, U6.3
- new net N$23: R29.2, U5.5
- new net N$25: Q1.1, R9.1
- new net N$29: C23.2, U5.6
- new net N$30: C18.1, Q1.11, Q1.7, Q1.8, Q1.9, R4.2, U2.A3
- new net N$32: C18.2, R9.2, U2.C2
- new net VBUS_OUT: C20.1, R29.1, SJ1.2, U5.10, U5.7, U5.8, VBUS_OUT_J.1
- new net VBUS_OUT_EN: U5.2
- new net VBUS_SENSE: C22.1, R26.1, R27.2
- net +3.8V: now also C6.1, R25.2, U6.1; no longer U4.5
- net GND: now also BAT_J.2, BAT_J2.2, C10.1, C11.1, C13.2, C14.2, C17.1, C19.2, C2.2, C20.2, C21.1, C22.2, C23.1, C24.1, C3.2, C4.2, C5.2, C6.2, C7.2, C8.2, C9.1, EXT_TH_J.2, PIO_J.2, R13.1, R14.1, R19.2, R27.1, R28.1, R5.1, R7.1, U1.7, U2.A2, U3.7, U4.7, U5.4, U6.2, USB_C.27, USB_C.28, USB_C.29, USB_C.30, USB_C.A1, USB_C.A12, USB_C.B1, USB_C.B12, VBUS_OUT_J.2; no longer R1.2
- net MCU_INT: now also PIO_J.1
- net MCU_SCL: no longer R21.1
- net MCU_SDA: now also R21.1
- net N$10: now also Q1.4, R10.1; no longer C18.2, Q1.2, Q2.2, R9.1
- net N$15: now also Q1.2, Q1.3; no longer Q1.4, Q2.4, R10.1
- net N$18: now also EXT_TH_J.1, R30.1; no longer EXT_TH_J.2
- net N$28: now also R20.1, R7.2, U3.6; no longer R8.1, U3.5
- net VBAT: now also BAT_J2.1, C24.2, R30.2
- net VBUS: now also C19.1, Q1.10, Q1.12, Q1.5, Q1.6, R20.2, R26.2, R8.1, SJ1.1, U5.1, U5.9; no longer D2.1, J1.1, Q1.3, Q2.3, R20.1, R8.2
- net VDD: no longer C15.2, R11.2, R21.2, R22.2, U$1.PAD_PU11, U$1.PAD_PU12, U$1.PAD_PU13, U$1.PAD_PU14, U$1.PAD_PU15, U$1.PAD_PU16, U$1.PAD_PU17, U$1.PAD_PU18, U$1.PAD_PU19, U$1.PAD_PU20, U4.1, U4.2
Routing:
- net GND: track 92.6 -> 0.00 mm, vias 32 -> 0
- net VDD: track 85.3 -> 0.00 mm, vias 5 -> 0
- net VSSA: track 78.3 -> 0.00 mm, vias 43 -> 0
- net VBUS: track 32.3 -> 0.00 mm, vias 9 -> 0
- net MCU_SDA: track 31.1 -> 0.00 mm, vias 1 -> 0
- net USART2_RX: track 27.2 -> 0.00 mm, vias 2 -> 0
- net MCU_SCL: track 27.1 -> 0.00 mm, vias 1 -> 0
- net USART2_TX: track 24.3 -> 0.00 mm, vias 1 -> 0
- net MCU_INT: track 23.8 -> 0.00 mm, vias 1 -> 0
- net USART5_TX: track 16.3 -> 0.00 mm, vias 1 -> 0
- net USART5_RX: track 15.5 -> 0.00 mm
- net USART1_TX: track 15.1 -> 0.00 mm, vias 1 -> 0
- net N$8: track 15.0 -> 0.00 mm, vias 1 -> 0
- net BAT_SDA: track 14.6 -> 0.00 mm
- net USART1_RX: track 14.4 -> 0.00 mm
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- removed copper zone on layer 1, net +3.8V
- removed copper zone on layer 16, net CSP
- removed copper zone on layer 1, net GND
- removed copper zone on layer 16, net GND
- removed copper zone on layer 1, net N$13
- removed copper zone on layer 1, net N$14
- removed copper zone on layer 16, net N$4
- removed copper zone on layer 16, net N$9
- removed copper zone on layer 16, net VBAT
- removed copper zone on layer 1, net VBUS
- removed copper zone on layer 16, net VBUS
- removed copper zone on layer 1, net VDD
- removed copper zone on layer 16, net VDD
- removed copper zone on layer 16, net VDDA
- removed copper zone on layer 1, net VSSA
- removed copper zone on layer 16, net VSSA
Other:
- board text removed: "+"
- board text removed: "+P"
- board text removed: "-"
- board text removed: "-P"

Commit message: -New Version (1b), reviewed and finished - adding the charging detection & current measurement circuit
Parts:
- removed L1: DFE252012P-1R0M=P2, HEXABITZ_RCLS:DFE2HCAH1R0MJ0L
- removed USB_C: 12401610E4#2A, HEXABITZ_CONNECTION_PARTS:12401610E42A
- added C25, C26, C27, C31: 100nF, HEXABITZ_RCLS:C-0603
- added C28, C29, C30: 1uF, HEXABITZ_RCLS:C-0805
- added C32: 22uF, HEXABITZ_RCLS:C-0805
- added D2: TL431QDBZR,215, HEXABITZ_RCLS:SOT23_TO-236AB_NEX
- added D5, D6, D7: CUS10S30,H3F, HEXABITZ_RCLS:1SS357TPH3F
- added J1: 12401610E4#2A12401610E42A, HEXABITZ_CONNECTION_PARTS:AMPHENOL_12401610E4_2A
- added R1: 10 mR, HEXABITZ_RCLS:R-0805
- added R31: 20K, HEXABITZ_RCLS:R-0603
- added R32: 27K, HEXABITZ_RCLS:R-0603
- added R33: 2K, HEXABITZ_RCLS:R-0603
- added R34: 100K, HEXABITZ_RCLS:R-0603
- added R35, R36: 22K, HEXABITZ_RCLS:R-0603
- added R37, R39: 10K, HEXABITZ_RCLS:R-0603
- added R38: 1M, HEXABITZ_RCLS:R-0603
- added SJ3: (no value), HEXABITZ_USER_INTERFACE_PARTS:SJ
- C10: value 47uF -> 33nF
- C11, C15: device HEXABITZ_RCLS:C-0603 -> HEXABITZ_RCLS:C-0805
- C16: value 22pF -> 33nF
- C24: value 22nF -> 100nF
- C8: device HEXABITZ_RCLS:T491B -> HEXABITZ_RCLS:C-0805
- C9: value 22uF -> 1nF
- R20, R8: value 100K -> 49.9K
- R25, R28: value 100K -> 220K
- R26: value 4.7K -> 47K
- R27: value 4.7K -> 20K
- R30: value 0R -> 100R
- R4: value 5 mR -> 1K; device HEXABITZ_RCLS:R-0805 -> HEXABITZ_RCLS:R-0603
- R5: value 33K -> 3mR; device HEXABITZ_RCLS:R-0603 -> HEXABITZ_RCLS:R1206
- R6: value 220K -> 1K
- R7: value 100K -> 1K
- SJ1, SJ2: device jumper:SJ -> HEXABITZ_USER_INTERFACE_PARTS:SJ
- U3: value TPS631000DRLR -> TSV772IQ2T; device HEXABITZ_ICs:TPS631000DRLR_TEX -> HEXABITZ_ICs:SON50P200X200X60-9N
- moved PIO_J 284.2 mm to (6.19, 19.7), turned to 210 degrees
- moved VBUS_OUT_J 278.3 mm to (16.2, 21.3), turned to 150 degrees
- moved C24 269.8 mm to (17.8, -3.65), flipped to the bottom, turned to 150 degrees
- moved C23 257.3 mm to (12.7, 11.6), flipped to the bottom, turned to 90 degrees
- moved R30 255.0 mm to (21.1, 2.70), flipped to the bottom, turned to 180 degrees
- moved R29 253.1 mm to (14.3, 11.6), flipped to the bottom, turned to 270 degrees
- moved C16 228.0 mm to (17.1, 13.8), turned to 180 degrees
- moved U4 226.6 mm to (-3.17, 5.87), flipped to the bottom
- moved C10 225.4 mm to (14.3, 8.57), turned to 180 degrees
- moved R8 222.7 mm to (17.1, 12.9), turned to 180 degrees
- moved R7 222.2 mm to (17.1, 11.3)
- moved C11 220.6 mm to (-3.97, 8.41), flipped to the bottom
- moved C15 217.6 mm to (0.00, 5.56), flipped to the bottom, turned to 90 degrees
- moved R20 216.1 mm to (14.3, 7.62), turned to 180 degrees
- moved R5 215.2 mm to (17.1, 1.69), flipped to the bottom, turned to 240 degrees
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Connections:
- net BAT_ALRT renamed N$15
- net N$2 renamed IND_LED
- removed net +3.8V: C10.2, C11.2, C16.1, C6.1, R25.2, R6.1, U3.1, U4.6, U6.1
- removed net BAT_SCL: R15.2, U2.B5
- removed net BAT_SDA: R17.2, U2.C5
- removed net N$13 (its old number): L1.1, U3.3
- removed net N$18 (its old number): EXT_TH_J.1, R13.2, R30.1, U2.A1
- removed net USART5_RX: U$1.PAD_PD1, U1.40
- removed net USART5_TX: U$1.PAD_PU1, U1.41
- removed net VDD: D4.2, FB1.2
- new net 3V3_OUT_PG: R39.1, U1.25, U4.4
- new net CHARGER_CURRENT_SENSE: C10.2, R20.2, U1.19, U3.1
- new net CHARGER_DETECT: D5.2, R38.2, U3.7
- new net MCU_LDO_EN: D6.2, U1.21
- new net N$11: C9.2, R6.2, U2.A3
- new net N$12: C18.1, Q1.11, Q1.7, Q1.8, Q1.9, R5.1, R6.1
- new net N$24: R15.2, U2.C5
- new net N$32: D5.1, D6.1, D7.1, R35.1
- new net N$35: D7.2, SJ3.1
- new net N$4: C30.2, R37.2, U5.2
- new net USART4_RX: U$1.PAD_PD1, U1.12
- new net USART4_TX: U$1.PAD_PU1, U1.11
- new net VBUS1: C26.2, R31.1, R32.2, R38.1, U3.5
- new net VBUS2: C27.2, D2.1, D2.2, R33.1, R34.2, U3.6
- new net VCHARGER: C25.2, C31.2, C8.1, J1.A4, J1.A9, J1.B4, J1.B9, R1.1, R7.2, U3.8
- new net VREF: C4.1, C5.1, U1.5
- net 3V3_OUT_EN: now also R36.1, U1.24; no longer R28.2, U4.5
- net GND: now also C16.1, C25.1, C26.1, C27.1, C28.1, C29.1, C30.1, C31.1, C32.2, D2.3, J1.A1, J1.A12, J1.B1, J1.B12, J1.S1, J1.S2, J1.S3, J1.S4, R25.2, R32.1, R34.1, R8.1, U3.4, U3.9; no longer C10.1, R5.1, R7.1, U1.24, U1.25, U3.7, USB_C.27, USB_C.28, USB_C.29, USB_C.30, USB_C.A1, USB_C.A12, USB_C.B1, USB_C.B12
- net MCU_3V3: now also D4.2, FB1.2, R39.2
- net MCU_INT: now also U1.16; no longer U1.19
- net MCU_SCL: now also R21.1
- net MCU_SDA: no longer R21.1
- net N$14: now also C10.1, R20.1, R4.1; no longer L1.2
- net N$16: now also R17.2, U2.B5; no longer R8.2, U3.5
- net N$17: now also R13.2, R30.1; no longer R14.2, R23.1
- net N$22: now also C28.2, R35.2
- net N$27: now also R7.1, R8.2, U3.3; no longer R5.2, R6.2, U3.8
- net N$28: now also EXT_TH_J.1, R14.2, R23.1, U2.A1; no longer R20.1, R7.2, U3.6
- net N$30: now also C29.2, R28.2, R36.2, U4.5; no longer C18.1, Q1.11, Q1.7, Q1.8, Q1.9, R4.2, U2.A3
- net STATUS_LED: now also U1.28; no longer U1.43
- net USART1_RX: now also U$1.PAD_PD4; no longer U$1.PAD_PD5
- net USART1_TX: now also U$1.PAD_PU4; no longer U$1.PAD_PU5
- net USART3_RX: now also U$1.PAD_PD3; no longer U$1.PAD_PD4
- net USART3_TX: now also U$1.PAD_PU3; no longer U$1.PAD_PU4
- net USART6_RX: now also U$1.PAD_PD5, U1.48; no longer U$1.PAD_PD3, U1.16
- net USART6_TX: now also U$1.PAD_PU5, U1.47; no longer U$1.PAD_PU3, U1.15
- net VBAT: now also C32.1, R23.2, R5.2; no longer R30.2, R4.1
- net VBUS: now also C11.2, C6.1, R1.2, R30.2, R31.2, R33.2, R4.2, SJ3.2, U4.6, U6.1; no longer C8.1, C9.2, R20.2, R23.2, R8.1, U3.4, USB_C.A4, USB_C.A9, USB_C.B4, USB_C.B9
- net VBUS_OUT_EN: now also R37.1, U1.15; no longer U5.2
- net VBUS_SENSE: now also U1.20
- net VDDA: no longer C4.1, C5.1, U1.4, U1.5
Routing:
- net GND: track 0.00 -> 256.6 mm, vias 0 -> 34
- net 3V3_OUT: track 0.00 -> 210.9 mm, vias 0 -> 13
- net MCU_3V3: track 0.00 -> 68.2 mm, vias 0 -> 4
- net VBUS: track 0.00 -> 60.8 mm, vias 0 -> 5
- net VBUS_OUT_EN: track 0.00 -> 36.6 mm, vias 0 -> 2
- net CHARGER_CURRENT_SENSE: track 0.00 -> 31.5 mm, vias 0 -> 2
- net MCU_INT: track 0.00 -> 29.9 mm, vias 0 -> 1
- net VBAT: track 0.00 -> 29.5 mm, vias 0 -> 1
- net CHARGER_DETECT: track 0.00 -> 25.2 mm, vias 0 -> 2
- net VBUS_SENSE: track 0.00 -> 21.3 mm
- net MCU_SCL: track 0.00 -> 19.7 mm, vias 0 -> 1
- net MCU_SDA: track 0.00 -> 19.7 mm, vias 0 -> 1
- net N$28: track 0.00 -> 18.4 mm, vias 0 -> 1
- net VCHARGER: track 0.00 -> 15.1 mm, vias 0 -> 8
- net USART3_TX: track 0.00 -> 15.0 mm, vias 0 -> 1
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- added copper zone on layer 16, net 3V3_OUT
- added copper zone on layer 1, net GND
- added copper zone on layer 15, net GND
- added copper zone on layer 16, net GND
- added copper zone on layer 2, net GND
- added copper zone on layer 16, net N$12
- added copper zone on layer 16, net N$13
- added copper zone on layer 16, net VBAT
- added copper zone on layer 16, net VBUS
- added copper zone on layer 16, net VBUS_OUT
- added copper zone on layer 1, net VCHARGER
- added copper zone on layer 16, net VCHARGER
Other:
- board text added: "+Vbus"
- board text added: "10A Max"
- board text added: "3V3/1A"
- board text added: "4.9V Max"
- board text added: "Charger_IN"
- board text added: "P4*"
- board text added: "P5"
- board text added: "Vbus_Out"
- board text removed: "*"
- board text removed: "3V3/2A"
- board text removed: "4.9 V MAX"
- board text removed: "P4"
- board text removed: "P5*"
